Commit message: pick and place

File: manipulator_description/urdf/manipulator.urdf (robot description, URDF)
Before this commit: robot manipulator_assembly_to_URDF_v2, 7 links, 6 joints
Joints:
- joint joint_1: limit (none) -> lower=-3.14 upper=3.14 effort=1000 velocity=1000; type continuous -> revolute
- joint joint_2: limit (none) -> lower=-1.5 upper=1.5 effort=1000 velocity=1000; type continuous -> revolute
- joint joint_3: limit (none) -> lower=-2.0 upper=1.2 effort=1000 velocity=1000; type continuous -> revolute
- joint joint_4: limit (none) -> lower=-1.57 upper=1.57 effort=1000 velocity=1000; type continuous -> revolute
